File: Robocat Pin.kicad_sch (KiCad schematic)
At the start: 17 parts, among them SW1 DP3T Switch, U1 555 Integrated Circuit

Commit message: Fixed footprints, parts, pcb
Parts:
- D1, D2: footprint Custom Library:1.3x3.2mm LED -> Custom Library:1206 LED; LCSC C3646934 -> C559121
- R1, R2, R3, R4, R5, R6: LCSC C4355165 -> C22962
- U1: LCSC C5160086 -> C543060
Changed lines of the file:
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@@
     (property "Reference" "D1" (id 0) (at 145.0975 81.28 0))
     (property "Value" "Blue LED" (id 1) (at 145.0975 83.82 0))
-    (property "Footprint" "Custom Library:1.3x3.2mm LED" (id 2) (at 143.51 88.9 0)
-      (effects (font (size 1.27 1.27)) hide)
-    )
-    (property "Datasheet" "https://www.lcsc.com/product-detail/Light-Emitting-Diodes-LED_EKINGLUX-E6CC1205RQBC2UDA_C2802678.html" (id 3) (at 143.51 88.9 0)
-      (effects (font (size 1.27 1.27)) hide)
-    )
-    (property "LCSC" "C3646934" (id 5) (at 143.51 88.9 0)
+    (property "Footprint" "Custom Library:1206 LED" (id 2) (at 143.51 88.9 0)
+      (effects (font (size 1.27 1.27)) hide)
+    )
+    (property "Datasheet" "https://www.lcsc.com/product-detail/Light-Emitting-Diodes-LED_MEIHUA-MHT151UBCT_C559121.html" (id 3) (at 143.51 88.9 0)
+      (effects (font (size 1.27 1.27)) hide)
+    )
+    (property "LCSC" "C559121" (id 5) (at 143.51 88.9 0)
       (effects (font (size 1.27 1.27)) hide)
     )
@@
       (effects (font (size 1.27 1.27)) hide)
     )
-    (property "LCSC" "C4355165" (id 5) (at 132.08 118.11 0)
+    (property "LCSC" "C22962" (id 5) (at 132.08 118.11 0)
       (effects (font (size 1.27 1.27)) hide)
     )
@@
       (effects (font (size 1.27 1.27)) hide)
     )
-    (property "LCSC" "C5160086" (id 5) (at 109.22 99.06 0)
+    (property "LCSC" "C543060" (id 5) (at 109.22 99.06 0)
       (effects (font (size 1.27 1.27)) hide)
     )
@@
       (effects (font (size 1.27 1.27)) hide)
     )
-    (property "LCSC" "C4355165" (id 4) (at 135.89 88.9 90)
+    (property "LCSC" "C22962" (id 4) (at 135.89 88.9 90)
       (effects (font (size 1.27 1.27)) hide)
     )
@@
     (property "Reference" "D2" (id 0) (at 145.0975 90.17 0))
     (property "Value" "Blue LED" (id 1) (at 145.0975 92.71 0))
-    (property "Footprint" "Custom Library:1.3x3.2mm LED" (id 2) (at 143.51 97.79 0)
-      (effects (font (size 1.27 1.27)) hide)
-    )
-    (property "Datasheet" "https://www.lcsc.com/product-detail/Light-Emitting-Diodes-LED_EKINGLUX-E6CC1205RQBC2UDA_C2802678.html" (id 3) (at 143.51 97.79 0)
-      (effects (font (size 1.27 1.27)) hide)
-    )
-    (property "LCSC" "C3646934" (id 5) (at 143.51 97.79 0)
+    (property "Footprint" "Custom Library:1206 LED" (id 2) (at 143.51 97.79 0)
+      (effects (font (size 1.27 1.27)) hide)
+    )
+    (property "Datasheet" "https://www.lcsc.com/product-detail/Light-Emitting-Diodes-LED_MEIHUA-MHT151UBCT_C559121.html" (id 3) (at 143.51 97.79 0)
+      (effects (font (size 1.27 1.27)) hide)
+    )
+    (property "LCSC" "C559121" (id 5) (at 143.51 97.79 0)
       (effects (font (size 1.27 1.27)) hide)
     )
@@
       (effects (font (size 1.27 1.27)) hide)
     )
-    (property "LCSC" "C4355165" (id 5) (at 135.89 97.79 0)
+    (property "LCSC" "C22962" (id 5) (at 135.89 97.79 0)
       (effects (font (size 1.27 1.27)) hide)
     )
@@
       (effects (font (size 1.27 1.27)) hide)
     )
-    (property "LCSC" "C4355165" (id 5) (at 123.19 87.63 0)
+    (property "LCSC" "C22962" (id 5) (at 123.19 87.63 0)
       (effects (font (size 1.27 1.27)) hide)
     )
@@
       (effects (font (size 1.27 1.27)) hide)
     )
-    (property "LCSC" "C4355165" (id 5) (at 127 110.49 0)
+    (property "LCSC" "C22962" (id 5) (at 127 110.49 0)
       (effects (font (size 1.27 1.27)) hide)
     )
@@
       (effects (font (size 1.27 1.27)) hide)
     )
-    (property "LCSC" "C4355165" (id 5) (at 127 118.11 0)
+    (property "LCSC" "C22962" (id 5) (at 127 118.11 0)
       (effects (font (size 1.27 1.27)) hide)
     )
@@
     )
     (path "/7f35b2a4-c774-457e-b5c9-0e4e4dac493a"
-      (reference "D1") (unit 1) (value "Blue LED") (footprint "Custom Library:1.3x3.2mm LED")
+      (reference "D1") (unit 1) (value "Blue LED") (footprint "Custom Library:1206 LED")
     )
     (path "/a96120e9-d7bd-4936-9b8e-1051e9751107"
-      (reference "D2") (unit 1) (value "Blue LED") (footprint "Custom Library:1.3x3.2mm LED")
+      (reference "D2") (unit 1) (value "Blue LED") (footprint "Custom Library:1206 LED")
     )
     (path "/e0cdf44c-3ee0-432d-ac41-707d8e8f7e04"

Commit message: Fixed issue that prevented it from blinking, cleaned up PCB design
Connections:
- net at C2.1, C3.1, C4.1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: now also SW1.6
- no-connect marks 2 -> 1
